Commit message: beautified the simulation a bit

File: src/robot_model/urdf/differential_1.xacro (robot description, xacro)
@@ -26,5 +26,5 @@
   </material>
   <gazebo reference="base_link_1">
-    <material>Gazebo/Orange</material>
+    <material>Gazebo/Green</material>
   </gazebo>
   <gazebo reference="link_left_wheel_1">
